File: 7segment.kicad_sch (KiCad schematic)
At the start: 12 parts, among them U2 74HC595BQ

Commit message: replace extended components with basic components.
Connections:
- no-connect marks 0 -> 1
Changed lines of the file:
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@@
 		(color 0 0 0 0)
+	)
+	(no_connect
+		(at 120.65 48.26)
 	)
 	(wire
